File: PNP.kicad_sch (KiCad schematic)
At the start: 13 parts, among them J4 Conn_01x06_Socket, J9 Screw_Terminal_01x02, U1 ESP32-S3-DevKitC, U10 Right Joystick, U6 Left Joystick

Commit message: Swap J4 to 2x06 header, drop KY-023 joysticks, rework TMC2209 daughterboard layout; add V0.2.0/V0.2.1 fab outputs
- PNP: J4 Conn_01x06 -> Conn_02x06 (PinHeader_2x06), removed Left/Right Joystick (U6/U10) from schematic and PCB, PCB re-routed (370 -> 366 segments area, vias 70 -> 58, zones 2 -> 1), ESP32-S3-DevKitC and MP1584EN footprints moved to Footprints lib, mask-to-copper clearance 0.005 mm
- TMC2209 daughterboard: PCB re-annotated/re-laid out (C5->C2, J6->J2, U8->U4, R7 removed)
- production/: PNP_V0.2.0 and V0.2.1 JLCPCB zips, BOM/CPL, netlist.ipc; fabrication-toolkit options
- code/: PlatformIO .gitignore and VS Code extension recommendations
Parts:
- removed U10: Right Joystick, Connector_JST:JST_XH_B5B-XH-A_1x05_P2.50mm_Vertical, symbol PNP:KY-023
- removed U6: Left Joystick, Connector_JST:JST_XH_B5B-XH-A_1x05_P2.50mm_Vertical, symbol PNP:KY-023
- J4: footprint Connector_PinHeader_2.54mm:PinHeader_1x06_P2.54mm_Vertical -> Connector_PinHeader_2.54mm:PinHeader_2x06_P2.54mm_Vertical; symbol Connector:Conn_01x06_Pin -> Connector_Generic:Conn_02x06_Counter_Clockwise
- U1: footprint Espressif:ESP32-S3-DevKitC -> Footprints:ESP32-S3-DevKitC
- U2: footprint PNP:Mini MP1584EN Buck Converter Module -> Footprints:Mini MP1584EN Buck Converter Module
Connections:
- net +3.3V: now also J4.12 (Pin_12); no longer J4.1 (Pin_1)
- net GND: now also J4.7 (Pin_7); no longer J4.6 (Pin_6)
- net GPIO0: now also J4.11 (Pin_11); no longer J4.2 (Pin_2)
- net GPIO11/ADC2_CH0: now also J4.9 (Pin_9); no longer J4.4 (Pin_4)
- net GPIO12/ADC2_CH1: now also J4.8 (Pin_8); no longer J4.5 (Pin_5)
- net GPIO15/ADC2_CH4/32K_P: now also J4.4 (Pin_4)
- net GPIO16/ADC2_CH5/32K_N: now also J4.2 (Pin_2)
- net GPIO17/ADC2_CH6: now also J4.1 (Pin_1)
- net GPIO3/ADC1_CH2: now also J4.10 (Pin_10); no longer J4.3 (Pin_3)
- net GPIO38: now also J4.6 (Pin_6)
- net GPIO45: now also J4.3 (Pin_3)
- net GPIO46: now also J4.5 (Pin_5)
